Commit message: lidar adjusted to proper position

File: gem_simulator/gem_description/urdf/gem_e4_main.urdf.xacro (robot description, xacro)
@@ -9,5 +9,5 @@
   <xacro:property name="velodyne_points" value="$(arg velodyne_points)" />
   <xacro:property name="laser_points" value="$(arg laser_points)" />
-  <xacro:include filename="$(find gem_description)/urdf/gem_e4.gazebo" />
+  <xacro:include filename="$(find gem_description)/urdf/gem.gazebo" />
   <xacro:include filename="$(find gem_description)/urdf/materials.xacro" />
   <xacro:include filename="$(find gem_description)/urdf/macros.xacro" />
@@ -971,6 +971,6 @@
   <xacro:steering_hinge_transmission name="right_steering_hinge" />
   <!-- *********************************************** Sensors ************************************************ -->
-  <xacro:VLP-16 parent="top_rack_link" name="velodyne" topic="/ouster/points" hz="10" samples="440" gpu="false" lasers="128" min_range="0.5" max_range="200.0" min_angle="-${M_PI}" max_angle="${M_PI}">
-    <origin xyz="0.02 0.42 0" rpy="1.5708 0 3.1416" />
+  <xacro:VLP-16 parent="top_rack_link" name="velodyne" topic="/velodyne_points" hz="10" samples="440" gpu="false">
+    <origin xyz="0.02 0.42 0" rpy="1.5708 0 3.1416" /> <!-- 1.5708 3.1416 -->
   </xacro:VLP-16>
   <!-- ************************* Front Camera ************************* -->
@@ -1131,31 +1131,4 @@
     <axis xyz="0 0 0" />
   </joint>
-  <!--
-  <link name="stereo_camera_link">
-    <collision>
-      <origin xyz="0 0 0" rpy="0 0 0"/>
-      <geometry>
-        <box size="0.05 0.05 0.05"/>
-      </geometry>
-    </collision>
-    <visual>
-      <origin xyz="0 0 0" rpy="0 0 0"/>
-      <geometry>
-        <box size="0.05 0.05 0.05"/>
-      </geometry>
-      <material name="red"/>
-    </visual>
-    <inertial>
-      <mass value="1e-5" />
-      <origin xyz="0 0 0" rpy="0 0 0"/>
-      <inertia ixx="1e-6" ixy="0" ixz="0" iyy="1e-6" iyz="0" izz="1e-6" />
-    </inertial>
-  </link>
-  <joint name="gem_stereo_camera_joint" type="fixed">
-    <origin xyz="-0.045 0 0" rpy="-1.5708 3.1416 0"/>
-    <parent link="front_camera_link"/>
-    <child link="stereo_camera_link"/>
-  </joint>
-  -->
   <!-- IMU -->
   <link name="IMU_link">
