Commit message: update urdf for control

File: gem_simulator/gem_description/urdf/gem_e4.urdf.xacro (robot description, xacro)
@@ -743,5 +743,5 @@
     <limit lower="-0.61" upper="0.61" effort="100" velocity="0.5" />
   </joint>
-  <link name="wheel_link_fl">
+  <link name="front_left_wheel_link">
     <inertial>
       <mass value="11" />
@@ -766,5 +766,5 @@
   <joint name="front_left_wheel_joint" type="continuous">
     <parent link="left_steering_hinge_link" />
-    <child link="wheel_link_fl" />
+    <child link="front_left_wheel_link" />
     <origin xyz="0 0 0" rpy="0 0 0" />
     <axis xyz="0 1 0" />
@@ -786,5 +786,5 @@
     <limit lower="-0.61" upper="0.61" effort="100" velocity="0.5" />
   </joint>
-  <link name="wheel_link_fr">
+  <link name="front_right_wheel_link">
     <inertial>
       <mass value="11" />
@@ -809,5 +809,5 @@
   <joint name="front_right_wheel_joint" type="continuous">
     <parent link="right_steering_hinge_link" />
-    <child link="wheel_link_fr" />
+    <child link="front_right_wheel_link" />
     <origin xyz="0 0 0" rpy="0 0 0" />
     <axis xyz="0 1 0" />
@@ -815,5 +815,5 @@
   </joint>
   <!-- ************************************ Rear Left Wheel ************************************ -->
-  <link name="wheel_link_rl">
+  <link name="rear_left_wheel_link">
     <inertial>
       <mass value="11" />
@@ -839,10 +839,10 @@
     <origin xyz="-1.2904 0.6545 0.027" rpy="0 0 0" />
     <parent link="base_link" />
-    <child link="wheel_link_rl" />
+    <child link="rear_left_wheel_link" />
     <axis xyz="0 1 0" />
     <limit effort="1000.0" velocity="100.0" />
   </joint>
   <!-- *********************************** Rear Right Wheel *********************************** -->
-  <link name="wheel_link_rr">
+  <link name="rear_right_wheel_link">
     <inertial>
       <mass value="11" />
@@ -868,11 +868,9 @@
     <origin xyz="-1.2904 -0.6535 0.027" rpy="0 0 0" />
     <parent link="base_link" />
-    <child link="wheel_link_rr" />
+    <child link="rear_right_wheel_link" />
     <axis xyz="0 1 0" />
     <limit effort="1000.0" velocity="100.0" />
   </joint>
   <!-- **************************************************************************************** -->
-  <klampt use_vis_geom="1" default_acc_max="4" default_vel_max="2">
-  </klampt>
   <!-- ******************************************** Transmissions ********************************************* -->
   <xacro:wheel_transmission name="rear_left_wheel" />

Commit message: Fix e4 gazebo materials

File: gem_simulator/gem_description/urdf/gem_e4.urdf.xacro (robot description, xacro)
@@ -32,5 +32,5 @@
         <mesh filename="package://gem_description/meshes/e4/base_link.STL" />
       </geometry>
-      <material name="">
+      <material name="blue">
         <color rgba="0 0 1 1" />
       </material>
@@ -43,4 +43,7 @@
     </collision>
   </link>
+  <gazebo reference="base_link">
+    <material>Gazebo/Blue</material>
+  </gazebo>
   <joint name="base_link" type="fixed">
     <origin xyz="0 0 0.268" rpy="0 0 0" />
@@ -74,4 +77,7 @@
     </collision>
   </link>
+  <gazebo reference="top_rack_link">
+    <material>Gazebo/Black</material>
+  </gazebo>
   <joint name="top_rack_joint" type="fixed">
     <origin xyz="-0.17 0 1.66" rpy="1.5708 0 0" />
@@ -104,4 +110,7 @@
     </collision>
   </link>
+  <gazebo reference="front_rack_link">
+    <material>Gazebo/Black</material>
+  </gazebo>
   <joint name="front_rack_joint" type="fixed">
     <origin xyz="1.7594 0 -0.15" rpy="1.5708 0 1.5708" />
@@ -134,4 +143,7 @@
     </collision>
   </link>
+  <gazebo reference="rear_rack_link">
+    <material>Gazebo/Black</material>
+  </gazebo>
   <joint name="rear_rack_joint" type="fixed">
     <origin xyz="-1.7372 0 -0.1" rpy="1.5708 0 -1.5708" />
@@ -164,4 +176,7 @@
     </collision>
   </link>
+  <gazebo reference="headlight_fr_link">
+    <material>Gazebo/White</material>
+  </gazebo>
   <joint name="headlight_fr_joint" type="fixed">
     <origin xyz="1.1677 -0.5 0.765" rpy="0 0 0" />
@@ -194,4 +209,7 @@
     </collision>
   </link>
+  <gazebo reference="headlight_fl_link">
+    <material>Gazebo/White</material>
+  </gazebo>
   <joint name="headlight_fl_joint" type="fixed">
     <origin xyz="1.1677 0.5 0.765" rpy="0 0 0" />
@@ -224,4 +242,7 @@
     </collision>
   </link>
+  <gazebo reference="turnlight_fl_link">
+    <material>Gazebo/Orange</material>
+  </gazebo>
   <joint name="turnlight_fl_joint" type="fixed">
     <origin xyz="1.1731 0.345 0.765" rpy="0 0 0" />
@@ -254,4 +275,7 @@
     </collision>
   </link>
+  <gazebo reference="turnlight_fr_link">
+    <material>Gazebo/Orange</material>
+  </gazebo>
   <joint name="turnlight_fr_joint" type="fixed">
     <origin xyz="1.1731 -0.345 0.765" rpy="0 0 0" />
@@ -284,4 +308,7 @@
     </collision>
   </link>
+  <gazebo reference="lightbar_link">
+    <material>Gazebo/Red</material>
+  </gazebo>
   <joint name="lightbar_joint" type="fixed">
     <origin xyz="-1.07655 0 0.9449" rpy="-1.9138 0 1.5708" />
@@ -315,4 +342,7 @@
     </collision>
   </link>
+  <gazebo reference="rear_left_stop_light_link">
+    <material>Gazebo/White</material>
+  </gazebo>
   <joint name="stoplight_rl_joint" type="fixed">
     <origin xyz="-1.625 0.38 0.423" rpy="0 0 3.1416" />
@@ -345,4 +375,7 @@
     </collision>
   </link>
+  <gazebo reference="rear_right_stop_light_link">
+    <material>Gazebo/White</material>
+  </gazebo>
   <joint name="stoplight_rr_joint" type="fixed">
     <origin xyz="-1.625 -0.38 0.423" rpy="0 0 3.1416" />
@@ -375,4 +408,7 @@
     </collision>
   </link>
+  <gazebo reference="taillight_rl_link">
+    <material>Gazebo/Red</material>
+  </gazebo>
   <joint name="taillight_rl_joint" type="fixed">
     <origin xyz="-1.62 0.32 0.203" rpy="0 0 3.1416" />
@@ -405,4 +441,7 @@
     </collision>
   </link>
+  <gazebo reference="taillight_rr_link">
+    <material>Gazebo/Red</material>
+  </gazebo>
   <joint name="taillight_rr_joint" type="fixed">
     <origin xyz="-1.62 -0.32 0.203" rpy="0 0 3.1416" />
@@ -435,4 +474,7 @@
     </collision>
   </link>
+  <gazebo reference="i_logo_fl_link">
+    <material>Gazebo/Orange</material>
+  </gazebo>
   <joint name="i_logo_fl_joint" type="fixed">
     <origin xyz="0.3966 0.6695 0.4123" rpy="0 0 0" />
@@ -465,4 +507,7 @@
     </collision>
   </link>
+  <gazebo reference="i_logo_rl_link">
+    <material>Gazebo/Orange</material>
+  </gazebo>
   <joint name="i_logo_rl_joint" type="fixed">
     <origin xyz="-0.42344 0.6695 0.4123" rpy="0 0 0" />
@@ -495,4 +540,7 @@
     </collision>
   </link>
+  <gazebo reference="i_logo_fr_link">
+    <material>Gazebo/Orange</material>
+  </gazebo>
   <joint name="i_logo_fr_joint" type="fixed">
     <origin xyz="0.3966 -0.68 0.4123" rpy="0 0 0" />
@@ -525,4 +573,7 @@
     </collision>
   </link>
+  <gazebo reference="i_logo_rr_link">
+    <material>Gazebo/Orange</material>
+  </gazebo>
   <joint name="i_logo_rr_joint" type="fixed">
     <origin xyz="-0.42344 -0.68 0.4123" rpy="0 0 0" />
@@ -554,4 +605,7 @@
     </collision>
   </link>
+  <gazebo reference="gps_antenna_main_link">
+    <material>Gazebo/White</material>
+  </gazebo>
   <joint name="gps_antenna_main_joint" type="fixed">
     <origin xyz="-0.01144 0.6525 1.7" rpy="0 0 0" />
@@ -582,4 +636,7 @@
     </collision>
   </link>
+  <gazebo reference="gps_antenna_aux_link">
+    <material>Gazebo/White</material>
+  </gazebo>
   <joint name="gps_antenna_aux_joint" type="fixed">
     <origin xyz="-0.01144 -0.6525 1.7" rpy="0 0 0" />
@@ -610,4 +667,7 @@
     </collision>
   </link>
+  <gazebo reference="top_lidar_link">
+    <material>Gazebo/White</material>
+  </gazebo>
   <joint name="top_lidar_joint" type="fixed">
     <origin xyz="-0.15144 0 2.08" rpy="0 0 0" />
@@ -638,4 +698,7 @@
     </collision>
   </link>
+  <gazebo reference="front_camera_link">
+    <material>Gazebo/White</material>
+  </gazebo>
   <joint name="front_camera_joint" type="fixed">
     <origin xyz="0.535 0 1.683" rpy="0 1.5708 0" />
@@ -666,4 +729,7 @@
     </collision>
   </link>
+  <gazebo reference="front_lidar_link">
+    <material>Gazebo/White</material>
+  </gazebo>
   <joint name="front_lidar_joint" type="fixed">
     <origin xyz="0.38206 0 1.71" rpy="0 0 0" />
@@ -694,4 +760,7 @@
     </collision>
   </link>
+  <gazebo reference="front_radar_link">
+    <material>Gazebo/White</material>
+  </gazebo>
   <joint name="front_radar_joint" type="fixed">
     <origin xyz="1.835 0 0.35" rpy="0 0 0" />
@@ -722,4 +791,7 @@
     </collision>
   </link>
+  <gazebo reference="imu_link">
+    <material>Gazebo/White</material>
+  </gazebo>
   <joint name="imu_joint" type="fixed">
     <origin xyz="-0.0044387 0 0.18294" rpy="0 0 0" />
@@ -736,4 +808,7 @@
     </inertial>
   </link>
+  <gazebo reference="left_steering_hinge_link">
+    <material>Gazebo/White</material>
+  </gazebo>
   <joint name="left_steering_hinge_joint" type="revolute">
     <parent link="base_link" />
@@ -764,4 +839,7 @@
     </collision>
   </link>
+  <gazebo reference="front_left_wheel_link">
+    <material>Gazebo/Black</material>
+  </gazebo>
   <joint name="front_left_wheel_joint" type="continuous">
     <parent link="left_steering_hinge_link" />
@@ -779,4 +857,7 @@
     </inertial>
   </link>
+  <gazebo reference="right_steering_hinge_link">
+    <material>Gazebo/White</material>
+  </gazebo>
   <joint name="right_steering_hinge_joint" type="revolute">
     <parent link="base_link" />
@@ -807,4 +888,7 @@
     </collision>
   </link>
+  <gazebo reference="front_right_wheel_link">
+    <material>Gazebo/Black</material>
+  </gazebo>
   <joint name="front_right_wheel_joint" type="continuous">
     <parent link="right_steering_hinge_link" />
@@ -836,4 +920,7 @@
     </collision>
   </link>
+  <gazebo reference="rear_left_wheel_link">
+    <material>Gazebo/Black</material>
+  </gazebo>
   <joint name="rear_left_wheel_joint" type="continuous">
     <origin xyz="-1.2904 0.6545 0.027" rpy="0 0 0" />
@@ -865,4 +952,7 @@
     </collision>
   </link>
+  <gazebo reference="rear_right_wheel_link">
+    <material>Gazebo/Black</material>
+  </gazebo>
   <joint name="rear_right_wheel_joint" type="continuous">
     <origin xyz="-1.2904 -0.6535 0.027" rpy="0 0 0" />
@@ -905,4 +995,7 @@
     </inertial>
   </link>
+  <gazebo reference="front_single_camera_link">
+    <material>Gazebo/White</material>
+  </gazebo>
   <!--
   <joint name="gem_front_camera_joint" type="fixed">
@@ -968,4 +1061,7 @@
     </inertial>
   </link>
+  <gazebo reference="IMU_link">
+    <material>Gazebo/White</material>
+  </gazebo>
   <joint name="IMU_joint" type="fixed">
     <origin xyz="-0.246 0 0.05" rpy="0 0 -1.5708"/>
@@ -997,4 +1093,7 @@
     </inertial>
   </link>
+  <gazebo reference="GPS_link">
+    <material>Gazebo/White</material>
+  </gazebo>
   <joint name="GPS_joint" type="fixed">
     <origin xyz="-0.246 0 0.05" rpy="0 0 0"/>
@@ -1023,4 +1122,7 @@
     </collision>
   </link>
+  <gazebo reference="front_sonar_link">
+    <material>Gazebo/Orange</material>
+  </gazebo>
   <joint name="front_sonar_joint" type="fixed">
     <origin xyz="0 0.38 0.065" rpy="0 -1.5708 -1.5708"/>
@@ -1049,4 +1151,7 @@
     </collision>
   </link>
+  <gazebo reference="rear_sonar_link">
+    <material>Gazebo/Orange</material>
+  </gazebo>
   <joint name="rear_sonar_joint" type="fixed">
     <origin xyz="0 0.38 0.065" rpy="0 -1.5708 -1.5708"/>

Commit message: Built and exported the actor_collision plugin and edited the highbay world file

File: gem_simulator/gem_description/urdf/gem_e4.urdf.xacro (robot description, xacro)
@@ -234,5 +234,5 @@
       </material>
     </visual>
-    <collision>
+    <collision>sc
       <origin xyz="0 0 0" rpy="0 0 0" />
       <geometry>

Commit message: Typo

File: gem_simulator/gem_description/urdf/gem_e4.urdf.xacro (robot description, xacro)
@@ -234,5 +234,5 @@
       </material>
     </visual>
-    <collision>sc
+    <collision>
       <origin xyz="0 0 0" rpy="0 0 0" />
       <geometry>

Commit message: add 4 corner cameras in e4

File: gem_simulator/gem_description/urdf/gem_e4.urdf.xacro (robot description, xacro)
@@ -1010,6 +1010,7 @@
     <child link="front_single_camera_link"/>
   </joint>
-  <!--
-  <link name="stereo_camera_link">
+  <!-- ************************* Corner Cameras ************************* -->
+  <!-- Front Left Corner Camera -->
+  <link name="front_left_corner_camera_link">
     <collision>
       <origin xyz="0 0 0" rpy="0 0 0"/>
@@ -1031,10 +1032,103 @@
     </inertial>
   </link>
-  <joint name="gem_stereo_camera_joint" type="fixed">
-    <origin xyz="-0.045 0 0" rpy="-1.5708 3.1416 0"/>
-    <parent link="front_camera_link"/>
-    <child link="stereo_camera_link"/>
-  </joint>
-  -->
+  <gazebo reference="front_left_corner_camera_link">
+    <material>Gazebo/Red</material>
+  </gazebo>
+  <joint name="front_left_corner_camera_joint" type="fixed">
+    <origin xyz="0.6 0.165 -0.597" rpy="-1.57 0 0"/>
+    <parent link="top_rack_link"/>
+    <child link="front_left_corner_camera_link"/>
+    <axis xyz="0 0 0" />
+  </joint>
+  <!-- Front Right Corner Camera -->
+  <link name="front_right_corner_camera_link">
+    <collision>
+      <origin xyz="0 0 0" rpy="0 0 0"/>
+      <geometry>
+        <box size="0.05 0.05 0.05"/>
+      </geometry>
+    </collision>
+    <visual>
+      <origin xyz="0 0 0" rpy="0 0 0"/>
+      <geometry>
+        <box size="0.05 0.05 0.05"/>
+      </geometry>
+      <material name="green"/>
+    </visual>
+    <inertial>
+      <mass value="1e-5" />
+      <origin xyz="0 0 0" rpy="0 0 0"/>
+      <inertia ixx="1e-6" ixy="0" ixz="0" iyy="1e-6" iyz="0" izz="1e-6" />
+    </inertial>
+  </link>
+  <gazebo reference="front_right_corner_camera_link">
+    <material>Gazebo/Green</material>
+  </gazebo>
+  <joint name="front_right_corner_camera_joint" type="fixed">
+    <origin xyz="0.6 0.165 0.58" rpy="-1.57 0 0"/>
+    <parent link="top_rack_link"/>
+    <child link="front_right_corner_camera_link"/>
+    <axis xyz="0 0 0" />
+  </joint>
+  <!-- Rear Left Corner Camera -->
+  <link name="rear_left_corner_camera_link">
+    <collision>
+      <origin xyz="0 0 0" rpy="0 0 0"/>
+      <geometry>
+        <box size="0.05 0.05 0.05"/>
+      </geometry>
+    </collision>
+    <visual>
+      <origin xyz="0 0 0" rpy="0 0 0"/>
+      <geometry>
+        <box size="0.05 0.05 0.05"/>
+      </geometry>
+      <material name="blue"/>
+    </visual>
+    <inertial>
+      <mass value="1e-5" />
+      <origin xyz="0 0 0" rpy="0 0 0"/>
+      <inertia ixx="1e-6" ixy="0" ixz="0" iyy="1e-6" iyz="0" izz="1e-6" />
+    </inertial>
+  </link>
+  <gazebo reference="rear_left_corner_camera_link">
+    <material>Gazebo/Blue</material>
+  </gazebo>
+  <joint name="rear_left_corner_camera_joint" type="fixed">
+    <origin xyz="-0.908 0.165 0.597" rpy="-1.57 3.14 0"/>
+    <parent link="top_rack_link"/>
+    <child link="rear_left_corner_camera_link"/>
+    <axis xyz="0 0 0" />
+  </joint>
+  <!-- Rear Right Corner Camera -->
+  <link name="rear_right_corner_camera_link">
+    <collision>
+      <origin xyz="0 0 0" rpy="0 0 0"/>
+      <geometry>
+        <box size="0.05 0.05 0.05"/>
+      </geometry>
+    </collision>
+    <visual>
+      <origin xyz="0 0 0" rpy="0 0 0"/>
+      <geometry>
+        <box size="0.05 0.05 0.05"/>
+      </geometry>
+      <material name="yellow"/>
+    </visual>
+    <inertial>
+      <mass value="1e-5" />
+      <origin xyz="0 0 0" rpy="0 0 0"/>
+      <inertia ixx="1e-6" ixy="0" ixz="0" iyy="1e-6" iyz="0" izz="1e-6" />
+    </inertial>
+  </link>
+  <gazebo reference="rear_right_corner_camera_link">
+    <material>Gazebo/Yellow</material>
+  </gazebo>
+  <joint name="rear_right_corner_camera_joint" type="fixed">
+    <origin xyz="-0.899 0.165 -0.597" rpy="-1.57 3.14 0"/>
+    <parent link="top_rack_link"/>
+    <child link="rear_right_corner_camera_link"/>
+    <axis xyz="0 0 0" />
+  </joint>
   <!-- IMU -->
   <link name="IMU_link">

Commit message: fix corner camera position and orientation

File: gem_simulator/gem_description/urdf/gem_e4.urdf.xacro (robot description, xacro)
@@ -1036,6 +1036,6 @@
   </gazebo>
   <joint name="front_left_corner_camera_joint" type="fixed">
-    <origin xyz="0.6 0.165 -0.597" rpy="-1.57 0 0"/>
-    <parent link="top_rack_link"/>
+    <origin xyz="0.5 0.6545 1.8" rpy="0 0.785 0.785"/>
+    <parent link="base_link"/>
     <child link="front_left_corner_camera_link"/>
     <axis xyz="0 0 0" />
@@ -1066,6 +1066,6 @@
   </gazebo>
   <joint name="front_right_corner_camera_joint" type="fixed">
-    <origin xyz="0.6 0.165 0.58" rpy="-1.57 0 0"/>
-    <parent link="top_rack_link"/>
+    <origin xyz="0.5 -0.6535 1.8" rpy="0 0.785 -0.785"/>
+    <parent link="base_link"/>
     <child link="front_right_corner_camera_link"/>
     <axis xyz="0 0 0" />
@@ -1096,6 +1096,6 @@
   </gazebo>
   <joint name="rear_left_corner_camera_joint" type="fixed">
-    <origin xyz="-0.908 0.165 0.597" rpy="-1.57 3.14 0"/>
-    <parent link="top_rack_link"/>
+    <origin xyz="-1.0 0.6545 1.8" rpy="0 0.785 2.356"/>
+    <parent link="base_link"/>
     <child link="rear_left_corner_camera_link"/>
     <axis xyz="0 0 0" />
@@ -1126,6 +1126,6 @@
   </gazebo>
   <joint name="rear_right_corner_camera_joint" type="fixed">
-    <origin xyz="-0.899 0.165 -0.597" rpy="-1.57 3.14 0"/>
-    <parent link="top_rack_link"/>
+    <origin xyz="-1.0 -0.6535 1.8" rpy="0 0.785 -2.356"/>
+    <parent link="base_link"/>
     <child link="rear_right_corner_camera_link"/>
     <axis xyz="0 0 0" />

Commit message: fixed top lidar

File: gem_simulator/gem_description/urdf/gem_e4.urdf.xacro (robot description, xacro)
@@ -971,6 +971,6 @@
   <xacro:steering_hinge_transmission name="right_steering_hinge" />
   <!-- *********************************************** Sensors ************************************************ -->
-  <xacro:VLP-16 parent="top_rack_link" name="velodyne" topic="/velodyne_points" hz="10" samples="440" gpu="false">
-    <origin xyz="0.02 0.42 0" rpy="1.5708 0 3.1416" /> <!-- 1.5708 3.1416 -->
+  <xacro:VLP-16 parent="top_rack_link" name="velodyne" topic="/velodyne_points" hz="10" samples="440" gpu="false" lasers="128" min_range="0.5" max_range="200.0" min_angle="-${M_PI}" max_angle="${M_PI}">
+    <origin xyz="0.02 0.25 0" rpy="1.5708 3.1416 3.1416" />
   </xacro:VLP-16>
   <!-- ************************* Front Camera ************************* -->

File: ros_drivers/velodyne_simulator/velodyne_description/urdf/VLP-16.urdf.xacro (robot description, xacro)
@@ -2,5 +2,5 @@
 <robot xmlns:xacro="http://www.ros.org/wiki/xacro" name="VLP-16">
   <xacro:property name="M_PI" value="3.1415926535897931" />
-  <xacro:macro name="VLP-16" params="*origin parent:=base_link name:=velodyne topic:=/velodyne_points hz:=10 lasers:=16 samples:=1875 collision_range:=0.3 min_range:=0.9 max_range:=130.0 noise:=0.008 min_angle:=-${M_PI} max_angle:=${M_PI} gpu:=false">
+  <xacro:macro name="VLP-16" params="*origin parent:=base_link name:=velodyne topic:=/velodyne_points hz:=10 lasers:=128 samples:=2048 collision_range:=0.3 min_range:=0.5 max_range:=200.0 noise:=0.001 min_angle:=-${M_PI} max_angle:=${M_PI} gpu:=false">
     <joint name="${name}_base_mount_joint" type="fixed">
       <xacro:insert_block name="origin" />
@@ -69,6 +69,6 @@
                 <samples>${lasers}</samples>
                 <resolution>1</resolution>
-                <min_angle>-${15.0*M_PI/180.0}</min_angle>
-                <max_angle> ${15.0*M_PI/180.0}</max_angle>
+                <min_angle>-${22.5*M_PI/180.0}</min_angle>
+                <max_angle>${22.5*M_PI/180.0}</max_angle>
               </vertical>
             </scan>
@@ -81,5 +81,5 @@
               <type>gaussian</type>
               <mean>0.0</mean>
-              <stddev>0.0</stddev>
+              <stddev>0.001</stddev>
             </noise>
           </ray>
@@ -109,6 +109,6 @@
                 <samples>${lasers}</samples>
                 <resolution>1</resolution>
-                <min_angle>-${15.0*M_PI/180.0}</min_angle>
-                <max_angle> ${15.0*M_PI/180.0}</max_angle>
+                <min_angle>-${22.5*M_PI/180.0}</min_angle>
+                <max_angle>${22.5*M_PI/180.0}</max_angle>
               </vertical>
             </scan>
@@ -121,5 +121,5 @@
               <type>gaussian</type>
               <mean>0.0</mean>
-              <stddev>0.0</stddev>
+              <stddev>0.001</stddev>
             </noise>
           </ray>

Commit message: added gem_e4.gazebo for e4 changes specifically

File: gem_simulator/gem_description/urdf/gem_e4.urdf.xacro (robot description, xacro)
@@ -9,5 +9,5 @@
   <xacro:property name="velodyne_points" value="$(arg velodyne_points)" />
   <xacro:property name="laser_points" value="$(arg laser_points)" />
-  <xacro:include filename="$(find gem_description)/urdf/gem.gazebo" />
+  <xacro:include filename="$(find gem_description)/urdf/gem_e4.gazebo" />
   <xacro:include filename="$(find gem_description)/urdf/materials.xacro" />
   <xacro:include filename="$(find gem_description)/urdf/macros.xacro" />
@@ -972,5 +972,5 @@
   <!-- *********************************************** Sensors ************************************************ -->
   <xacro:VLP-16 parent="top_rack_link" name="velodyne" topic="/velodyne_points" hz="10" samples="440" gpu="false" lasers="128" min_range="0.5" max_range="200.0" min_angle="-${M_PI}" max_angle="${M_PI}">
-    <origin xyz="0.02 0.25 0" rpy="1.5708 3.1416 3.1416" />
+    <origin xyz="0.02 0.25 0" rpy="1.5708 0 3.1416" />
   </xacro:VLP-16>
   <!-- ************************* Front Camera ************************* -->
