Commit message: Matched Urdf to work with real car extrinsics

File: gem_simulator/gem_description/urdf/gem_e4.urdf.xacro (robot description, xacro)
@@ -9,5 +9,5 @@
   <xacro:property name="velodyne_points" value="$(arg velodyne_points)" />
   <xacro:property name="laser_points" value="$(arg laser_points)" />
-  <xacro:include filename="$(find gem_description)/urdf/gem.gazebo" />
+  <xacro:include filename="$(find gem_description)/urdf/gem_e4.gazebo" />
   <xacro:include filename="$(find gem_description)/urdf/materials.xacro" />
   <xacro:include filename="$(find gem_description)/urdf/macros.xacro" />
@@ -971,6 +971,6 @@
   <xacro:steering_hinge_transmission name="right_steering_hinge" />
   <!-- *********************************************** Sensors ************************************************ -->
-  <xacro:VLP-16 parent="top_rack_link" name="velodyne" topic="/velodyne_points" hz="10" samples="440" gpu="false">
-    <origin xyz="0.02 0.42 0" rpy="1.5708 0 3.1416" /> <!-- 1.5708 3.1416 -->
+  <xacro:VLP-16 parent="top_rack_link" name="velodyne" topic="/velodyne_points" hz="10" samples="440" gpu="false" lasers="128" min_range="0.5" max_range="200.0" min_angle="-${M_PI}" max_angle="${M_PI}">
+    <origin xyz="0.02 0.25 0" rpy="1.5708 0 3.1416" />
   </xacro:VLP-16>
   <!-- ************************* Front Camera ************************* -->
@@ -1010,7 +1010,6 @@
     <child link="front_single_camera_link"/>
   </joint>
-  <!-- ************************* Corner Cameras ************************* -->
-  <!-- Front Left Corner Camera -->
-  <link name="front_left_corner_camera_link">
+  <!--
+  <link name="stereo_camera_link">
     <collision>
       <origin xyz="0 0 0" rpy="0 0 0"/>
@@ -1032,103 +1031,10 @@
     </inertial>
   </link>
-  <gazebo reference="front_left_corner_camera_link">
-    <material>Gazebo/Red</material>
-  </gazebo>
-  <joint name="front_left_corner_camera_joint" type="fixed">
-    <origin xyz="0.5 0.6545 1.8" rpy="0 0.785 0.785"/>
-    <parent link="base_link"/>
-    <child link="front_left_corner_camera_link"/>
-    <axis xyz="0 0 0" />
-  </joint>
-  <!-- Front Right Corner Camera -->
-  <link name="front_right_corner_camera_link">
-    <collision>
-      <origin xyz="0 0 0" rpy="0 0 0"/>
-      <geometry>
-        <box size="0.05 0.05 0.05"/>
-      </geometry>
-    </collision>
-    <visual>
-      <origin xyz="0 0 0" rpy="0 0 0"/>
-      <geometry>
-        <box size="0.05 0.05 0.05"/>
-      </geometry>
-      <material name="green"/>
-    </visual>
-    <inertial>
-      <mass value="1e-5" />
-      <origin xyz="0 0 0" rpy="0 0 0"/>
-      <inertia ixx="1e-6" ixy="0" ixz="0" iyy="1e-6" iyz="0" izz="1e-6" />
-    </inertial>
-  </link>
-  <gazebo reference="front_right_corner_camera_link">
-    <material>Gazebo/Green</material>
-  </gazebo>
-  <joint name="front_right_corner_camera_joint" type="fixed">
-    <origin xyz="0.5 -0.6535 1.8" rpy="0 0.785 -0.785"/>
-    <parent link="base_link"/>
-    <child link="front_right_corner_camera_link"/>
-    <axis xyz="0 0 0" />
-  </joint>
-  <!-- Rear Left Corner Camera -->
-  <link name="rear_left_corner_camera_link">
-    <collision>
-      <origin xyz="0 0 0" rpy="0 0 0"/>
-      <geometry>
-        <box size="0.05 0.05 0.05"/>
-      </geometry>
-    </collision>
-    <visual>
-      <origin xyz="0 0 0" rpy="0 0 0"/>
-      <geometry>
-        <box size="0.05 0.05 0.05"/>
-      </geometry>
-      <material name="blue"/>
-    </visual>
-    <inertial>
-      <mass value="1e-5" />
-      <origin xyz="0 0 0" rpy="0 0 0"/>
-      <inertia ixx="1e-6" ixy="0" ixz="0" iyy="1e-6" iyz="0" izz="1e-6" />
-    </inertial>
-  </link>
-  <gazebo reference="rear_left_corner_camera_link">
-    <material>Gazebo/Blue</material>
-  </gazebo>
-  <joint name="rear_left_corner_camera_joint" type="fixed">
-    <origin xyz="-1.0 0.6545 1.8" rpy="0 0.785 2.356"/>
-    <parent link="base_link"/>
-    <child link="rear_left_corner_camera_link"/>
-    <axis xyz="0 0 0" />
-  </joint>
-  <!-- Rear Right Corner Camera -->
-  <link name="rear_right_corner_camera_link">
-    <collision>
-      <origin xyz="0 0 0" rpy="0 0 0"/>
-      <geometry>
-        <box size="0.05 0.05 0.05"/>
-      </geometry>
-    </collision>
-    <visual>
-      <origin xyz="0 0 0" rpy="0 0 0"/>
-      <geometry>
-        <box size="0.05 0.05 0.05"/>
-      </geometry>
-      <material name="yellow"/>
-    </visual>
-    <inertial>
-      <mass value="1e-5" />
-      <origin xyz="0 0 0" rpy="0 0 0"/>
-      <inertia ixx="1e-6" ixy="0" ixz="0" iyy="1e-6" iyz="0" izz="1e-6" />
-    </inertial>
-  </link>
-  <gazebo reference="rear_right_corner_camera_link">
-    <material>Gazebo/Yellow</material>
-  </gazebo>
-  <joint name="rear_right_corner_camera_joint" type="fixed">
-    <origin xyz="-1.0 -0.6535 1.8" rpy="0 0.785 -2.356"/>
-    <parent link="base_link"/>
-    <child link="rear_right_corner_camera_link"/>
-    <axis xyz="0 0 0" />
-  </joint>
+  <joint name="gem_stereo_camera_joint" type="fixed">
+    <origin xyz="-0.045 0 0" rpy="-1.5708 3.1416 0"/>
+    <parent link="front_camera_link"/>
+    <child link="stereo_camera_link"/>
+  </joint>
+  -->
   <!-- IMU -->
   <link name="IMU_link">

File: ros_drivers/velodyne_simulator/velodyne_description/urdf/VLP-16.urdf.xacro (robot description, xacro)
@@ -2,5 +2,5 @@
 <robot xmlns:xacro="http://www.ros.org/wiki/xacro" name="VLP-16">
   <xacro:property name="M_PI" value="3.1415926535897931" />
-  <xacro:macro name="VLP-16" params="*origin parent:=base_link name:=velodyne topic:=/velodyne_points hz:=10 lasers:=16 samples:=1875 collision_range:=0.3 min_range:=0.9 max_range:=130.0 noise:=0.008 min_angle:=-${M_PI} max_angle:=${M_PI} gpu:=false">
+  <xacro:macro name="VLP-16" params="*origin parent:=base_link name:=velodyne topic:=/velodyne_points hz:=10 lasers:=128 samples:=2048 collision_range:=0.3 min_range:=0.5 max_range:=200.0 noise:=0.001 min_angle:=-${M_PI} max_angle:=${M_PI} gpu:=false">
     <joint name="${name}_base_mount_joint" type="fixed">
       <xacro:insert_block name="origin" />
@@ -69,6 +69,6 @@
                 <samples>${lasers}</samples>
                 <resolution>1</resolution>
-                <min_angle>-${15.0*M_PI/180.0}</min_angle>
-                <max_angle> ${15.0*M_PI/180.0}</max_angle>
+                <min_angle>-${22.5*M_PI/180.0}</min_angle>
+                <max_angle>${22.5*M_PI/180.0}</max_angle>
               </vertical>
             </scan>
@@ -81,5 +81,5 @@
               <type>gaussian</type>
               <mean>0.0</mean>
-              <stddev>0.0</stddev>
+              <stddev>0.001</stddev>
             </noise>
           </ray>
@@ -109,6 +109,6 @@
                 <samples>${lasers}</samples>
                 <resolution>1</resolution>
-                <min_angle>-${15.0*M_PI/180.0}</min_angle>
-                <max_angle> ${15.0*M_PI/180.0}</max_angle>
+                <min_angle>-${22.5*M_PI/180.0}</min_angle>
+                <max_angle>${22.5*M_PI/180.0}</max_angle>
               </vertical>
             </scan>
@@ -121,5 +121,5 @@
               <type>gaussian</type>
               <mean>0.0</mean>
-              <stddev>0.0</stddev>
+              <stddev>0.001</stddev>
             </noise>
           </ray>

Commit message: Add OS1 file and add corresponding rviz configs

File: gem_simulator/gem_description/urdf/gem_e4.urdf.xacro (robot description, xacro)
@@ -12,5 +12,5 @@
   <xacro:include filename="$(find gem_description)/urdf/materials.xacro" />
   <xacro:include filename="$(find gem_description)/urdf/macros.xacro" />
-  <xacro:include filename="$(find velodyne_description)/urdf/VLP-16.urdf.xacro" />
+  <xacro:include filename="$(find velodyne_description)/urdf/OS1.urdf.xacro" />
   <link name="base_footprint">
   </link>
@@ -971,7 +971,7 @@
   <xacro:steering_hinge_transmission name="right_steering_hinge" />
   <!-- *********************************************** Sensors ************************************************ -->
-  <xacro:VLP-16 parent="top_rack_link" name="velodyne" topic="/ouster/points" hz="10" samples="440" gpu="false" lasers="128" min_range="0.5" max_range="200.0" min_angle="-${M_PI}" max_angle="${M_PI}">
+  <xacro:OS1 parent="top_rack_link" name="ouster" topic="/ouster/points" hz="10" samples="440" gpu="false" lasers="128" min_range="0.5" max_range="200.0" min_angle="-${M_PI}" max_angle="${M_PI}">
     <origin xyz="0.02 0.42 0" rpy="1.5708 0 3.1416" />
-  </xacro:VLP-16>
+  </xacro:OS1>
   <!-- ************************* Front Camera ************************* -->
   <link name="front_single_camera_link">

File: ros_drivers/velodyne_simulator/velodyne_description/urdf/OS1.urdf.xacro (robot description, xacro)
@@ -1,6 +1,6 @@
 <?xml version="1.0"?>
-<robot xmlns:xacro="http://www.ros.org/wiki/xacro" name="VLP-16">
+<robot xmlns:xacro="http://www.ros.org/wiki/xacro" name="OS1">
   <xacro:property name="M_PI" value="3.1415926535897931" />
-  <xacro:macro name="VLP-16" params="*origin parent:=base_link name:=velodyne topic:=/velodyne_points hz:=10 lasers:=16 samples:=1875 collision_range:=0.3 min_range:=0.9 max_range:=130.0 noise:=0.008 min_angle:=-${M_PI} max_angle:=${M_PI} gpu:=false">
+  <xacro:macro name="OS1" params="*origin parent:=base_link name:=velodyne topic:=/velodyne_points hz:=10 lasers:=128 samples:=2048 collision_range:=0.3 min_range:=0.5 max_range:=200.0 noise:=0.001 min_angle:=-${M_PI} max_angle:=${M_PI} gpu:=false">
     <joint name="${name}_base_mount_joint" type="fixed">
       <xacro:insert_block name="origin" />
@@ -54,5 +54,5 @@
     <gazebo reference="${name}">
       <xacro:if value="${gpu}">
-        <sensor type="gpu_ray" name="${name}-VLP16">
+        <sensor type="gpu_ray" name="${name}-OS1">
           <pose>0 0 0 0 0 0</pose>
           <visualize>false</visualize>
@@ -69,6 +69,6 @@
                 <samples>${lasers}</samples>
                 <resolution>1</resolution>
-                <min_angle>-${15.0*M_PI/180.0}</min_angle>
-                <max_angle> ${15.0*M_PI/180.0}</max_angle>
+                <min_angle>-${22.5*M_PI/180.0}</min_angle>
+                <max_angle>${22.5*M_PI/180.0}</max_angle>
               </vertical>
             </scan>
@@ -81,5 +81,5 @@
               <type>gaussian</type>
               <mean>0.0</mean>
-              <stddev>0.0</stddev>
+              <stddev>0.001</stddev>
             </noise>
           </ray>
@@ -94,5 +94,5 @@
       </xacro:if>
       <xacro:unless value="${gpu}">
-        <sensor type="ray" name="${name}-VLP16">
+        <sensor type="ray" name="${name}-OS1">
           <pose>0 0 0 0 0 0</pose>
           <visualize>false</visualize>
@@ -109,6 +109,6 @@
                 <samples>${lasers}</samples>
                 <resolution>1</resolution>
-                <min_angle>-${15.0*M_PI/180.0}</min_angle>
-                <max_angle> ${15.0*M_PI/180.0}</max_angle>
+                <min_angle>-${22.5*M_PI/180.0}</min_angle>
+                <max_angle>${22.5*M_PI/180.0}</max_angle>
               </vertical>
             </scan>
@@ -121,5 +121,5 @@
               <type>gaussian</type>
               <mean>0.0</mean>
-              <stddev>0.0</stddev>
+              <stddev>0.001</stddev>
             </noise>
           </ray>

Commit message: Fix corner camera position

File: gem_simulator/gem_description/urdf/gem_e4.urdf.xacro (robot description, xacro)
@@ -1013,14 +1013,14 @@
   <!-- Front Left Corner Camera -->
   <link name="front_left_corner_camera_link">
-    <collision>
-      <origin xyz="0 0 0" rpy="0 0 0"/>
-      <geometry>
-        <box size="0.05 0.05 0.05"/>
-      </geometry>
-    </collision>
-    <visual>
-      <origin xyz="0 0 0" rpy="0 0 0"/>
-      <geometry>
-        <box size="0.05 0.05 0.05"/>
+    <!-- <collision>
+      <origin xyz="0 0 0" rpy="0 0 0"/>
+      <geometry>
+        <box size="0.02 0.02 0.01"/>
+      </geometry>
+    </collision> -->
+    <visual>
+      <origin xyz="0 0 0" rpy="0 0 0"/>
+      <geometry>
+        <box size="0.02 0.02 0.01"/>
       </geometry>
       <material name="red"/>
@@ -1036,5 +1036,5 @@
   </gazebo>
   <joint name="front_left_corner_camera_joint" type="fixed">
-    <origin xyz="0.5 0.6545 1.8" rpy="0 0.785 0.785"/>
+    <origin xyz="0.5 0.6545 1.75" rpy="0 0.785 0.785"/>
     <parent link="base_link"/>
     <child link="front_left_corner_camera_link"/>
@@ -1043,14 +1043,14 @@
   <!-- Front Right Corner Camera -->
   <link name="front_right_corner_camera_link">
-    <collision>
-      <origin xyz="0 0 0" rpy="0 0 0"/>
-      <geometry>
-        <box size="0.05 0.05 0.05"/>
-      </geometry>
-    </collision>
-    <visual>
-      <origin xyz="0 0 0" rpy="0 0 0"/>
-      <geometry>
-        <box size="0.05 0.05 0.05"/>
+    <!-- <collision>
+      <origin xyz="0 0 0" rpy="0 0 0"/>
+      <geometry>
+        <box size="0.02 0.02 0.01"/>
+      </geometry>
+    </collision> -->
+    <visual>
+      <origin xyz="0 0 0" rpy="0 0 0"/>
+      <geometry>
+        <box size="0.02 0.02 0.01"/>
       </geometry>
       <material name="green"/>
@@ -1066,5 +1066,5 @@
   </gazebo>
   <joint name="front_right_corner_camera_joint" type="fixed">
-    <origin xyz="0.5 -0.6535 1.8" rpy="0 0.785 -0.785"/>
+    <origin xyz="0.5 -0.6535 1.75" rpy="0 0.785 -0.785"/>
     <parent link="base_link"/>
     <child link="front_right_corner_camera_link"/>
@@ -1073,14 +1073,14 @@
   <!-- Rear Left Corner Camera -->
   <link name="rear_left_corner_camera_link">
-    <collision>
-      <origin xyz="0 0 0" rpy="0 0 0"/>
-      <geometry>
-        <box size="0.05 0.05 0.05"/>
-      </geometry>
-    </collision>
-    <visual>
-      <origin xyz="0 0 0" rpy="0 0 0"/>
-      <geometry>
-        <box size="0.05 0.05 0.05"/>
+    <!-- <collision>
+      <origin xyz="0 0 0" rpy="0 0 0"/>
+      <geometry>
+        <box size="0.02 0.02 0.01"/>
+      </geometry>
+    </collision> -->
+    <visual>
+      <origin xyz="0 0 0" rpy="0 0 0"/>
+      <geometry>
+        <box size="0.02 0.02 0.01"/>
       </geometry>
       <material name="blue"/>
@@ -1096,5 +1096,5 @@
   </gazebo>
   <joint name="rear_left_corner_camera_joint" type="fixed">
-    <origin xyz="-1.0 0.6545 1.8" rpy="0 0.785 2.356"/>
+    <origin xyz="-1.0 0.6545 1.75" rpy="0 0.785 2.356"/>
     <parent link="base_link"/>
     <child link="rear_left_corner_camera_link"/>
@@ -1103,14 +1103,14 @@
   <!-- Rear Right Corner Camera -->
   <link name="rear_right_corner_camera_link">
-    <collision>
-      <origin xyz="0 0 0" rpy="0 0 0"/>
-      <geometry>
-        <box size="0.05 0.05 0.05"/>
-      </geometry>
-    </collision>
-    <visual>
-      <origin xyz="0 0 0" rpy="0 0 0"/>
-      <geometry>
-        <box size="0.05 0.05 0.05"/>
+    <!-- <collision>
+      <origin xyz="0 0 0" rpy="0 0 0"/>
+      <geometry>
+        <box size="0.02 0.02 0.01"/>
+      </geometry>
+    </collision> -->
+    <visual>
+      <origin xyz="0 0 0" rpy="0 0 0"/>
+      <geometry>
+        <box size="0.02 0.02 0.01"/>
       </geometry>
       <material name="yellow"/>
@@ -1126,5 +1126,5 @@
   </gazebo>
   <joint name="rear_right_corner_camera_joint" type="fixed">
-    <origin xyz="-1.0 -0.6535 1.8" rpy="0 0.785 -2.356"/>
+    <origin xyz="-1.0 -0.6535 1.75" rpy="0 0.785 -2.356"/>
     <parent link="base_link"/>
     <child link="rear_right_corner_camera_link"/>
