Commit message: Update GEM urdf to contain LiDAR

File: gem_simulator/gem_description/urdf/gem.urdf.xacro (robot description, xacro)
@@ -39,5 +39,5 @@
       <origin xyz="0 0 0" rpy="0 0 0" />
       <geometry>
-        <mesh filename="package://gem_description/meshes/base_link.STL" />
+        <mesh filename="file://$(find gem_description)/meshes/base_link.STL" />
       </geometry>
       <material name="white" />
@@ -46,5 +46,5 @@
       <origin xyz="0 0 0" rpy="0 0 0" />
       <geometry>
-        <mesh filename="package://gem_description/meshes/base_link.STL" />
+        <mesh filename="file://$(find gem_description)/meshes/base_link.STL" />
       </geometry>
     </collision>
@@ -71,5 +71,5 @@
       <origin xyz="0 0 0" rpy="0 0 0" />
       <geometry>
-        <mesh filename="package://gem_description/meshes/chair_link.STL" />
+        <mesh filename="file://$(find gem_description)/meshes/chair_link.STL" />
       </geometry>
       <material name="grey" />
@@ -78,5 +78,5 @@
       <origin xyz="0 0 0" rpy="0 0 0" />
       <geometry>
-        <mesh filename="package://gem_description/meshes/chair_link.STL" />
+        <mesh filename="file://$(find gem_description)/meshes/chair_link.STL" />
       </geometry>
     </collision>
@@ -103,5 +103,5 @@
       <origin xyz="0 0 0" rpy="0 0 0" />
       <geometry>
-        <mesh filename="package://gem_description/meshes/door_link.STL" />
+        <mesh filename="file://$(find gem_description)/meshes/door_link.STL" />
       </geometry>
       <material name="white" />
@@ -110,5 +110,5 @@
       <origin xyz="0 0 0" rpy="0 0 0" />
       <geometry>
-        <mesh filename="package://gem_description/meshes/door_link.STL" />
+        <mesh filename="file://$(find gem_description)/meshes/door_link.STL" />
       </geometry>
     </collision>
@@ -135,5 +135,5 @@
       <origin xyz="0 0 0" rpy="0 0 0" />
       <geometry>
-        <mesh filename="package://gem_description/meshes/top_rack_link.STL" />
+        <mesh filename="file://$(find gem_description)/meshes/top_rack_link.STL" />
       </geometry>
       <material name="black" />
@@ -142,5 +142,5 @@
       <origin xyz="0 0 0" rpy="0 0 0" />
       <geometry>
-        <mesh filename="package://gem_description/meshes/top_rack_link.STL" />
+        <mesh filename="file://$(find gem_description)/meshes/top_rack_link.STL" />
       </geometry>
     </collision>
@@ -167,5 +167,5 @@
       <origin xyz="0 0 0" rpy="0 0 0" />
       <geometry>
-        <mesh filename="package://gem_description/meshes/front_rack_link.STL" />
+        <mesh filename="file://$(find gem_description)/meshes/front_rack_link.STL" />
       </geometry>
       <material name="black" />
@@ -174,5 +174,5 @@
       <origin xyz="0 0 0" rpy="0 0 0" />
       <geometry>
-        <mesh filename="package://gem_description/meshes/front_rack_link.STL" />
+        <mesh filename="file://$(find gem_description)/meshes/front_rack_link.STL" />
       </geometry>
     </collision>
@@ -199,5 +199,5 @@
       <origin xyz="0 0 0" rpy="0 0 0" />
       <geometry>
-        <mesh filename="package://gem_description/meshes/rear_rack_link.STL" />
+        <mesh filename="file://$(find gem_description)/meshes/rear_rack_link.STL" />
       </geometry>
       <material name="black" />
@@ -206,5 +206,5 @@
       <origin xyz="0 0 0" rpy="0 0 0" />
       <geometry>
-        <mesh filename="package://gem_description/meshes/rear_rack_link.STL" />
+        <mesh filename="file://$(find gem_description)/meshes/rear_rack_link.STL" />
       </geometry>
     </collision>
@@ -231,5 +231,5 @@
       <origin xyz="0 0 0" rpy="0 0 0" />
       <geometry>
-        <mesh filename="package://gem_description/meshes/front_right_head_light_link.STL" />
+        <mesh filename="file://$(find gem_description)/meshes/front_right_head_light_link.STL" />
       </geometry>
       <material name="white" />
@@ -238,5 +238,5 @@
       <origin xyz="0 0 0" rpy="0 0 0" />
       <geometry>
-        <mesh filename="package://gem_description/meshes/front_right_head_light_link.STL" />
+        <mesh filename="file://$(find gem_description)/meshes/front_right_head_light_link.STL" />
       </geometry>
     </collision>
@@ -263,5 +263,5 @@
       <origin xyz="0 0 0" rpy="0 0 0" />
       <geometry>
-        <mesh filename="package://gem_description/meshes/front_left_head_light_link.STL" />
+        <mesh filename="file://$(find gem_description)/meshes/front_left_head_light_link.STL" />
       </geometry>
       <material name="white" />
@@ -270,5 +270,5 @@
       <origin xyz="0 0 0" rpy="0 0 0" />
       <geometry>
-        <mesh filename="package://gem_description/meshes/front_left_head_light_link.STL" />
+        <mesh filename="file://$(find gem_description)/meshes/front_left_head_light_link.STL" />
       </geometry>
     </collision>
@@ -295,5 +295,5 @@
       <origin xyz="0 0 0" rpy="0 0 0" />
       <geometry>
-        <mesh filename="package://gem_description/meshes/front_right_turn_light_link.STL" />
+        <mesh filename="file://$(find gem_description)/meshes/front_right_turn_light_link.STL" />
       </geometry>
       <material name="orange" />
@@ -302,5 +302,5 @@
       <origin xyz="0 0 0" rpy="0 0 0" />
       <geometry>
-        <mesh filename="package://gem_description/meshes/front_right_turn_light_link.STL" />
+        <mesh filename="file://$(find gem_description)/meshes/front_right_turn_light_link.STL" />
       </geometry>
     </collision>
@@ -327,5 +327,5 @@
       <origin xyz="0 0 0" rpy="0 0 0" />
       <geometry>
-        <mesh filename="package://gem_description/meshes/front_left_turn_light_link.STL" />
+        <mesh filename="file://$(find gem_description)/meshes/front_left_turn_light_link.STL" />
       </geometry>
       <material name="orange" />
@@ -334,5 +334,5 @@
       <origin xyz="0 0 0" rpy="0 0 0" />
       <geometry>
-        <mesh filename="package://gem_description/meshes/front_left_turn_light_link.STL" />
+        <mesh filename="file://$(find gem_description)/meshes/front_left_turn_light_link.STL" />
       </geometry>
     </collision>
@@ -359,5 +359,5 @@
       <origin xyz="0 0 0" rpy="0 0 0" />
       <geometry>
-        <mesh filename="package://gem_description/meshes/rear_right_light_link.STL" />
+        <mesh filename="file://$(find gem_description)/meshes/rear_right_light_link.STL" />
       </geometry>
       <material name="red" />
@@ -366,5 +366,5 @@
       <origin xyz="0 0 0" rpy="0 0 0" />
       <geometry>
-        <mesh filename="package://gem_description/meshes/rear_right_light_link.STL" />
+        <mesh filename="file://$(find gem_description)/meshes/rear_right_light_link.STL" />
       </geometry>
     </collision>
@@ -391,5 +391,5 @@
       <origin xyz="0 0 0" rpy="0 0 0" />
       <geometry>
-        <mesh filename="package://gem_description/meshes/rear_left_light_link.STL" />
+        <mesh filename="file://$(find gem_description)/meshes/rear_left_light_link.STL" />
       </geometry>
       <material name="red" />
@@ -398,5 +398,5 @@
       <origin xyz="0 0 0" rpy="0 0 0" />
       <geometry>
-        <mesh filename="package://gem_description/meshes/rear_left_light_link.STL" />
+        <mesh filename="file://$(find gem_description)/meshes/rear_left_light_link.STL" />
       </geometry>
     </collision>
@@ -423,5 +423,5 @@
       <origin xyz="0 0 0" rpy="0 0 0" />
       <geometry>
-        <mesh filename="package://gem_description/meshes/rear_left_stop_light_link.STL" />
+        <mesh filename="file://$(find gem_description)/meshes/rear_left_stop_light_link.STL" />
       </geometry>
       <material name="red" />
@@ -430,5 +430,5 @@
       <origin xyz="0 0 0" rpy="0 0 0" />
       <geometry>
-        <mesh filename="package://gem_description/meshes/rear_left_stop_light_link.STL" />
+        <mesh filename="file://$(find gem_description)/meshes/rear_left_stop_light_link.STL" />
       </geometry>
     </collision>
@@ -455,5 +455,5 @@
       <origin xyz="0 0 0" rpy="0 0 0" />
       <geometry>
-        <mesh filename="package://gem_description/meshes/rear_right_stop_light_link.STL" />
+        <mesh filename="file://$(find gem_description)/meshes/rear_right_stop_light_link.STL" />
       </geometry>
       <material name="red" />
@@ -462,5 +462,5 @@
       <origin xyz="0 0 0" rpy="0 0 0" />
       <geometry>
-        <mesh filename="package://gem_description/meshes/rear_right_stop_light_link.STL" />
+        <mesh filename="file://$(find gem_description)/meshes/rear_right_stop_light_link.STL" />
       </geometry>
     </collision>
@@ -487,5 +487,5 @@
       <origin xyz="0 0 0" rpy="0 0 0" />
       <geometry>
-        <mesh filename="package://gem_description/meshes/right_blue_outer_link.STL" />
+        <mesh filename="file://$(find gem_description)/meshes/right_blue_outer_link.STL" />
       </geometry>
       <material name="blue" />
@@ -494,5 +494,5 @@
       <origin xyz="0 0 0" rpy="0 0 0" />
       <geometry>
-        <mesh filename="package://gem_description/meshes/right_blue_outer_link.STL" />
+        <mesh filename="file://$(find gem_description)/meshes/right_blue_outer_link.STL" />
       </geometry>
     </collision>
@@ -519,5 +519,5 @@
       <origin xyz="0 0 0" rpy="0 0 0" />
       <geometry>
-        <mesh filename="package://gem_description/meshes/right_I_link.STL" />
+        <mesh filename="file://$(find gem_description)/meshes/right_I_link.STL" />
       </geometry>
       <material name="orange" />
@@ -526,5 +526,5 @@
       <origin xyz="0 0 0" rpy="0 0 0" />
       <geometry>
-        <mesh filename="package://gem_description/meshes/right_I_link.STL" />
+        <mesh filename="file://$(find gem_description)/meshes/right_I_link.STL" />
       </geometry>
     </collision>
@@ -551,5 +551,5 @@
       <origin xyz="0 0 0" rpy="0 0 0" />
       <geometry>
-        <mesh filename="package://gem_description/meshes/left_blue_outer_link.STL" />
+        <mesh filename="file://$(find gem_description)/meshes/left_blue_outer_link.STL" />
       </geometry>
       <material name="blue" />
@@ -558,5 +558,5 @@
       <origin xyz="0 0 0" rpy="0 0 0" />
       <geometry>
-        <mesh filename="package://gem_description/meshes/left_blue_outer_link.STL" />
+        <mesh filename="file://$(find gem_description)/meshes/left_blue_outer_link.STL" />
       </geometry>
     </collision>
@@ -583,5 +583,5 @@
       <origin xyz="0 0 0" rpy="0 0 0" />
       <geometry>
-        <mesh filename="package://gem_description/meshes/left_I_link.STL" />
+        <mesh filename="file://$(find gem_description)/meshes/left_I_link.STL" />
       </geometry>
       <material name="orange" />
@@ -590,5 +590,5 @@
       <origin xyz="0 0 0" rpy="0 0 0" />
       <geometry>
-        <mesh filename="package://gem_description/meshes/left_I_link.STL" />
+        <mesh filename="file://$(find gem_description)/meshes/left_I_link.STL" />
       </geometry>
     </collision>
@@ -615,5 +615,5 @@
       <origin xyz="0 0 0" rpy="0 0 0" />
       <geometry>
-        <mesh filename="package://gem_description/meshes/right_antenna_link.STL" />
+        <mesh filename="file://$(find gem_description)/meshes/right_antenna_link.STL" />
       </geometry>
       <material name="grey" />
@@ -622,5 +622,5 @@
       <origin xyz="0 0 0" rpy="0 0 0" />
       <geometry>
-        <mesh filename="package://gem_description/meshes/right_antenna_link.STL" />
+        <mesh filename="file://$(find gem_description)/meshes/right_antenna_link.STL" />
       </geometry>
     </collision>
@@ -647,5 +647,5 @@
       <origin xyz="0 0 0" rpy="0 0 0" />
       <geometry>
-        <mesh filename="package://gem_description/meshes/left_antenna_link.STL" />
+        <mesh filename="file://$(find gem_description)/meshes/left_antenna_link.STL" />
       </geometry>
       <material name="grey" />
@@ -654,5 +654,5 @@
       <origin xyz="0 0 0" rpy="0 0 0" />
       <geometry>
-        <mesh filename="package://gem_description/meshes/left_antenna_link.STL" />
+        <mesh filename="file://$(find gem_description)/meshes/left_antenna_link.STL" />
       </geometry>
     </collision>
@@ -679,5 +679,5 @@
       <origin xyz="0 0 0" rpy="0 0 0" />
       <geometry>
-        <mesh filename="package://gem_description/meshes/rear_left_emergency_button_link.STL" />
+        <mesh filename="file://$(find gem_description)/meshes/rear_left_emergency_button_link.STL" />
       </geometry>
       <material name="red" />
@@ -686,5 +686,5 @@
       <origin xyz="0 0 0" rpy="0 0 0" />
       <geometry>
-        <mesh filename="package://gem_description/meshes/rear_left_emergency_button_link.STL" />
+        <mesh filename="file://$(find gem_description)/meshes/rear_left_emergency_button_link.STL" />
       </geometry>
     </collision>
@@ -711,5 +711,5 @@
       <origin xyz="0 0 0" rpy="0 0 0" />
       <geometry>
-        <mesh filename="package://gem_description/meshes/rear_right_emergency_button_link.STL" />
+        <mesh filename="file://$(find gem_description)/meshes/rear_right_emergency_button_link.STL" />
       </geometry>
       <material name="red" />
@@ -718,5 +718,5 @@
       <origin xyz="0 0 0" rpy="0 0 0" />
       <geometry>
-        <mesh filename="package://gem_description/meshes/rear_right_emergency_button_link.STL" />
+        <mesh filename="file://$(find gem_description)/meshes/rear_right_emergency_button_link.STL" />
       </geometry>
     </collision>
@@ -743,5 +743,5 @@
       <origin xyz="0 0 0" rpy="0 0 0" />
       <geometry>
-        <mesh filename="package://gem_description/meshes/front_left_emergency_button_link.STL" />
+        <mesh filename="file://$(find gem_description)/meshes/front_left_emergency_button_link.STL" />
       </geometry>
       <material name="red" />
@@ -750,5 +750,5 @@
       <origin xyz="0 0 0" rpy="0 0 0" />
       <geometry>
-        <mesh filename="package://gem_description/meshes/front_left_emergency_button_link.STL" />
+        <mesh filename="file://$(find gem_description)/meshes/front_left_emergency_button_link.STL" />
       </geometry>
     </collision>
@@ -775,5 +775,5 @@
       <origin xyz="0 0 0" rpy="0 0 0" />
       <geometry>
-        <mesh filename="package://gem_description/meshes/front_right_emergency_button_link.STL" />
+        <mesh filename="file://$(find gem_description)/meshes/front_right_emergency_button_link.STL" />
       </geometry>
       <material name="red" />
@@ -782,5 +782,5 @@
       <origin xyz="0 0 0" rpy="0 0 0" />
       <geometry>
-        <mesh filename="package://gem_description/meshes/front_right_emergency_button_link.STL" />
+        <mesh filename="file://$(find gem_description)/meshes/front_right_emergency_button_link.STL" />
       </geometry>
     </collision>
@@ -801,5 +801,5 @@
       <origin xyz="0 0 0" rpy="0 0 0" />
       <geometry>
-        <mesh filename="package://gem_description/meshes/rear_light_bar_link.STL" />
+        <mesh filename="file://$(find gem_description)/meshes/rear_light_bar_link.STL" />
       </geometry>
       <material name="red" />
@@ -808,5 +808,5 @@
       <origin xyz="0 0 0" rpy="0 0 0" />
       <geometry>
-        <mesh filename="package://gem_description/meshes/rear_light_bar_link.STL" />
+        <mesh filename="file://$(find gem_description)/meshes/rear_light_bar_link.STL" />
       </geometry>
     </collision>
@@ -828,5 +828,5 @@
       <origin xyz="0 0 0" rpy="0 0 0" />
       <geometry>
-        <mesh filename="package://gem_description/meshes/front_camera_link.STL" />
+        <mesh filename="file://$(find gem_description)/meshes/front_camera_link.STL" />
       </geometry>
       <material name="black" />
@@ -835,5 +835,5 @@
       <origin xyz="0 0 0" rpy="0 0 0" />
       <geometry>
-        <mesh filename="package://gem_description/meshes/front_camera_link.STL" />
+        <mesh filename="file://$(find gem_description)/meshes/front_camera_link.STL" />
       </geometry>
     </collision>
@@ -877,5 +877,5 @@
       <origin xyz="0 0 0" rpy="0 0 0"/>
       <geometry>
-        <mesh filename="package://gem_description/meshes/front_left_wheel_link.STL"/>
+        <mesh filename="file://$(find gem_description)/meshes/front_left_wheel_link.STL"/>
       </geometry>
       <material name="black"/>
@@ -902,5 +902,5 @@
       <origin xyz="0 0 0" rpy="0 0 0"/>
       <geometry>
-        <mesh filename="package://gem_description/meshes/front_right_wheel_link.STL"/>
+        <mesh filename="file://$(find gem_description)/meshes/front_right_wheel_link.STL"/>
       </geometry>
       <material name="black" />
@@ -927,5 +927,5 @@
       <origin xyz="0 0 0" rpy="0 0 0"/>
       <geometry>
-        <mesh filename="package://gem_description/meshes/rear_left_wheel_link.STL"/>
+        <mesh filename="file://$(find gem_description)/meshes/rear_left_wheel_link.STL"/>
       </geometry>
       <material name="black"/>
@@ -952,5 +952,5 @@
       <origin xyz="0 0 0" rpy="0 0 0"/>
       <geometry>
-        <mesh filename="package://gem_description/meshes/rear_right_wheel_link.STL"/>
+        <mesh filename="file://$(find gem_description)/meshes/rear_right_wheel_link.STL"/>
       </geometry>
       <material name="black"/>
@@ -1019,37 +1019,9 @@
   <!-- *********************************************** Sensors ************************************************ -->
   <!-- ************************* Front Camera ************************* -->
-  <link name="front_single_camera_link">
-    <collision>
-      <origin xyz="0 0 0" rpy="0 0 0"/>
-      <geometry>
-        <box size="0.05 0.05 0.05"/>
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